File: m0ii0 alpha.kicad_pcb (KiCad board)
At the start: 2 copper layers, 200.2 x 86.4 mm, 121 parts, among them IC1 W25Q16JVUXIQ, J1 USB_C_Receptacle_USB2.0, SW1 boot, U1 RP2040, U2 USBLC6-2SC6, U3 XC6206PxxxMR-Regulator_Linear, Y1 12MHz

Commit message: added silkscreen
Parts:
- added G***: LOGO, LOGO, F.Cu at (121.4, 60.3)
- added G***: LOGO, LOGO, B.Cu at (34.1, 102.4)
Other:
- board text added: "Calvin0563"
- board text added: "JLCJLCJLCJLC"
- board text added: "alpha"
- board text added: "layout by patcoll"
- board text added: "m0ii0"
- board text added: "m0ii0 alpha"
- board text added: "pcb by"
